File: pcb/_autosave-binary_watch_dev_pcb.kicad_pcb (KiCad board)
At the start: 2 copper layers, 100 x 100 mm, 69 parts, among them K1 PWR_SELECT, M1 MNT, M2 MNT, M3 MNT, M4 MNT, P1 ISP, P2 USB-MICRO-B, P3 LED_ISENSE, P7 MCU_ISENSE, P8 TST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

Commit message: Add new dev pcb files from nightly build of kicad
Other:
- board size 100 x 100 mm -> 50 x 50 mm
Changed lines of the file:
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@@
     (area 99.924999 39.924999 200.075001 140.075001)
     (thickness 1.6)
-    (drawings 6)
+    (drawings 4)
     (tracks 464)
     (zones 0)
@@
       (net 48 /LED_SNSI_P))
   )
-  (gr_line (start 100 140) (end 100 40) (angle 90) (layer Edge.Cuts) (width 0.15))
+  (gr_line (start 100 140) (end 100 90) (angle 90) (layer Edge.Cuts) (width 0.15))
+  (gr_line (start 150 140) (end 100 140) (angle 90) (layer Edge.Cuts) (width 0.15))
   (gr_line (start 150 90) (end 100 90) (angle 90) (layer Edge.Cuts) (width 0.15))
   (gr_line (start 150 140) (end 150 90) (angle 90) (layer Edge.Cuts) (width 0.15))
-  (gr_line (start 200 40) (end 100 40) (angle 90) (layer Edge.Cuts) (width 0.15))
-  (gr_line (start 200 140) (end 100 140) (angle 90) (layer Edge.Cuts) (width 0.15))
-  (gr_line (start 200 40) (end 200 140) (angle 90) (layer Edge.Cuts) (width 0.15))
   (segment (start 125.4318 119.7498) (end 125.4318 117.9318) (width 0.508) (layer F.Cu) (net 1))
   (segment (start 125.4318 117.9318) (end 125.4 117.9) (width 0.508) (layer F.Cu) (net 1))
