File: pcb/binary_watch_dev_pcb.kicad_pcb (KiCad board)
At the start: 2 copper layers, 100 x 100 mm, 69 parts, among them K1 PWR_SELECT, M1 MNT, M2 MNT, M3 MNT, M4 MNT, P1 ISP, P2 USB-MICRO-B, P3 LED_ISENSE, P7 MCU_ISENSE, P8 TST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

Commit message: Finish dev schematic and layout, create gerbers to send to manufacture
Parts:
- added SW1A1: BUTTON_1, _ Custom Lib:EVQ-P7C01P, F.Cu at (115.0, 138.2)
- added SW2A1: BUTTON_2, _ Custom Lib:EVQ-P7C01P, F.Cu at (125.0, 138.2)
- added SYM: Symbol_OSHW-Logo_SilkScreen_07Jul2012, Symbols:Symbol_OSHW-Logo_SilkScreen, F.Cu at (111.2, 116.0)
- U3: footprint SMD_Packages:SOT-223 -> _ Custom Lib:SOT-223
Routing:
- net /MCU_SNSI_N: track 9.88 -> 0.88 mm
- net VCC: track 87.4 -> 96.4 mm
- net /SW_1: track 24.1 -> 32.4 mm
- net /SW_2: track 25.0 -> 33.3 mm
- net GND: track 87.8 -> 94.4 mm, vias 27 -> 31
- net /LED_SNSI_P: track 5.29 -> 0.48 mm
- net +BATT: track 86.4 -> 91.2 mm
- net +3.3V: track 120.3 -> 116.9 mm
Other:
- board size 100 x 100 mm -> 50 x 50 mm
- board text added: "A"
- board text added: "B"
- board text added: "Binary Watch"
- board text added: "Dev Rev A"
- board text added: "ISP"
- board text added: "LEDs"
- board text added: "Lee Szuba"
- board text added: "MCU"
- board text added: "Nov 2014"
- board text added: "RESET"
- board text added: "USB"
