File: pcb/binary_watch_pcb.sch (KiCad schematic (older format))
At the start: 37 parts, among them IC1 ATMEGA168PA-A, P1 CONN_3X2, SW1 SW_PUSH, SW2 SW_PUSH, X1 CRYSTAL

Commit message: Gen fab outputs, pdfs, and finish final routing.
Parts:
- removed C1: 1uF, ~, symbol C
- removed IC?: ATMEGA168PA-M, MLF/QFN32, symbol ATMEGA168PA-M
- removed SW1: SW_PUSH, ~, symbol SW_PUSH
- added BAT-N1: CONN_01X01, symbol CONN_01X01
- added C2: 1uF, Capacitors_SMD:C_0603, symbol C
- added R19: 10k, Resistors_SMD:R_0402, symbol R
- added SW1A1: BUTTON_1, _ Custom Lib:EVQ-P7C01P, symbol SW_PUSH
- BT1: footprint ~ -> _ Custom Lib:CR2032_MPD; Manufacturer P/N (none) -> BU2032SM-HD-G; Vendor P/N (none) -> BU2032SM-HD-GCT-ND
- C3, C4, C5: footprint ~ -> Capacitors_SMD:C_0603; Manufacturer P/N (none) -> LMK107B7105KA-T; Vendor P/N (none) -> 587-1242-1-ND
- C6, C7: value C -> 9pF; footprint ~ -> Capacitors_SMD:C_0402; Manufacturer P/N (none) -> GRM1555C1H9R0BA01D; Vendor P/N (none) -> 490-6257-1-ND
- DH10, DH11, DH7, DH8, DH9, DM1, DM2, DM3, DM4, DM5, DM6: footprint ~ -> LEDs:LED-0805
- P1: value CONN_3X2 -> ISP; footprint (none) -> Pin_Headers:Pin_Header_Straight_2x03
- R1, R10, R11, R12, R13, R2, R3, R4, R5, R6, R7, R8, R9: footprint ~ -> Resistors_SMD:R_0402
- SW2A1: renamed from SW2; value SW_PUSH -> BUTTON_2; footprint ~ -> _ Custom Lib:EVQ-P7C01P; Manufacturer P/N (none) -> EVQ-P7C01P; Vendor P/N (none) -> P16765CT-ND
- U1: renamed from IC1; footprint TQFP32 -> SMD_Packages:TQFP-32
- X1: value CRYSTAL -> 32.768kHz; footprint ~ -> _ Custom Lib:XTAL_ABS07; Manufacturer P/N (none) -> ABS07-32.768KHZ-9-T; Vendor P/N (none) -> 535-9544-1-ND
Connections:
- net labels added: +BATT
- net labels removed: +3.3V
- wire segments 170 -> 117
- no-connect marks 12 -> 6
Other:
- moved on the sheet: BT1, C3, C4, C5, P1, R12, R13, SW2A1
